File: LED_Control_RTC_version2.kicad_sch (KiCad schematic)
At the start: 4 parts

Commit message: Cleaned up messy reference numbering Added labels to schematic
Other:
- moved on the sheet: H1, H2, H3, H4
