File: LED_Control_RTC_version2.kicad_pcb (KiCad board)
At the start: 4 copper layers, 100 x 80 mm, 143 parts, among them J1 Screw_Terminal_01x02, J10 Conn_01x06_Male, J2 Conn_01x02, J3 Conn_02x04_Odd_Even, J4 DS1023-2*8SF11, J5 DS1023-2*8SF11, J6 Conn_01x03_Female, J7 Conn_ARM_JTAG_SWD_10, J8 Conn_ARM_JTAG_SWD_10, J9 Conn_01x06_Male, Q1 IRLR8726TRPBF, Q10 IRLR8726TRPBF, Q11 PJM2309PSA, Q2 IRLR8726TRPBF, Q3 IRLR8726TRPBF, Q4 IRLR8726TRPBF, Q5 IRLR8726TRPBF, Q6 IRLR8726TRPBF, Q7 IRLR8726TRPBF, Q8 IRLR8726TRPBF, Q9 IRLR8726TRPBF, U1 STM32F103C8Tx, U101 TC4427, U102 TC4427, U103 TC4427, U104 TC4427, U105 TC4427, U2 STM32G030C6Tx, U3 AT24C16D-XHM-B, U4 MAX3485, U5 TPS5401, U6 LM1117-3.3, Y1 16MHz, Y2 32.768KHz

Commit message: Ready for prod
Other:
- board text added: "JLCJLCJLCJLC"
Changed lines of the file:
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@@
       (outputformat 1)
       (mirror false)
-      (drillshape 1)
+      (drillshape 0)
       (scaleselection 1)
-      (outputdirectory "")
+      (outputdirectory "gerbers/")
     )
   )
@@
     (fp_line (start -7.1 -3) (end -7.1 3) (layer "F.Fab") (width 0.1))
     (fp_line (start -2.8 -4.75) (end -0.8 -4.75) (layer "F.Fab") (width 0.1))
-    (pad "1" thru_hole roundrect (at 0 0 180) (size 1.8 3.6) (drill 1.2) (layers *.Cu *.Mask) (roundrect_rratio 0.138889)
+    (pad "1" thru_hole roundrect (at 0 0 180) (size 1.8 3.6) (drill 1.2) (layers *.Cu *.Mask) (roundrect_rratio 0.1388888889)
       (net 8 "/MCUs + Peripherals/OUT1") (pinfunction "Pin_1") (pintype "passive"))
     (pad "2" thru_hole oval (at 3.81 0 180) (size 1.8 3.6) (drill 1.2) (layers *.Cu *.Mask)
@@
     (fp_line (start -1.6 0.8) (end -1.6 -0.8) (layer "F.Fab") (width 0.1))
     (fp_line (start -1.6 -0.8) (end 1.6 -0.8) (layer "F.Fab") (width 0.1))
-    (pad "1" smd roundrect (at -1.4625 0 270) (size 1.125 1.75) (layers "F.Cu" "F.Paste" "F.Mask") (roundrect_rratio 0.222222)
+    (pad "1" smd roundrect (at -1.4625 0 270) (size 1.125 1.75) (layers "F.Cu" "F.Paste" "F.Mask") (roundrect_rratio 0.2222222222)
       (net 29 "+5V") (pintype "passive"))
-    (pad "2" smd roundrect (at 1.4625 0 270) (size 1.125 1.75) (layers "F.Cu" "F.Paste" "F.Mask") (roundrect_rratio 0.222222)
+    (pad "2" smd roundrect (at 1.4625 0 270) (size 1.125 1.75) (layers "F.Cu" "F.Paste" "F.Mask") (roundrect_rratio 0.2222222222)
       (net 2 "GND") (pintype "passive"))
     (model "${KICAD6_3DMODEL_DIR}/Resistor_SMD.3dshapes/R_1206_3216Metric.wrl"
@@
     (fp_line (start 2.25 -1.6) (end 2.25 1.6) (layer "F.Fab") (width 0.1))
     (fp_line (start 2.25 1.6) (end -2.25 1.6) (layer "F.Fab") (width 0.1))
-    (pad "1" smd roundrect (at -2.1375 0 90) (size 1.125 3.4) (layers "F.Cu" "F.Paste" "F.Mask") (roundrect_rratio 0.222222)
+    (pad "1" smd roundrect (at -2.1375 0 90) (size 1.125 3.4) (layers "F.Cu" "F.Paste" "F.Mask") (roundrect_rratio 0.2222222222)
       (net 60 "/Power Delivery/Power_IN") (pintype "passive"))
-    (pad "2" smd roundrect (at 2.1375 0 90) (size 1.125 3.4) (layers "F.Cu" "F.Paste" "F.Mask") (roundrect_rratio 0.222222)
+    (pad "2" smd roundrect (at 2.1375 0 90) (size 1.125 3.4) (layers "F.Cu" "F.Paste" "F.Mask") (roundrect_rratio 0.2222222222)
       (net 33 "Net-(F2-Pad2)") (pintype "passive"))
     (model "${KICAD6_3DMODEL_DIR}/Fuse.3dshapes/Fuse_1812_4532Metric.wrl"
@@
     (fp_line (start -7.1 3) (end 26.15 3) (layer "F.Fab") (width 0.1))
     (fp_line (start -2.8 -3.5) (end -2.8 -4.75) (layer "F.Fab") (width 0.1))
-    (pad "1" thru_hole roundrect (at 0 0 180) (size 1.8 3.6) (drill 1.2) (layers *.Cu *.Mask) (roundrect_rratio 0.138889)
+    (pad "1" thru_hole roundrect (at 0 0 180) (size 1.8 3.6) (drill 1.2) (layers *.Cu *.Mask) (roundrect_rratio 0.1388888889)
       (net 19 "/MCUs + Peripherals/OUT6") (pinfunction "Pin_1") (pintype "passive"))
     (pad "2" thru_hole oval (at 3.81 0 180) (size 1.8 3.6) (drill 1.2) (layers *.Cu *.Mask)
@@
     (fp_line (start -7.1 -1.2) (end -7.1 8) (layer "F.Fab") (width 0.1))
     (fp_line (start 0 0) (end -0.8 -1.2) (layer "F.Fab") (width 0.1))
-    (pad "1" thru_hole roundrect (at 0 0) (size 1.8 3.6) (drill 1.2) (layers *.Cu *.Mask) (roundrect_rratio 0.138889)
+    (pad "1" thru_hole roundrect (at 0 0) (size 1.8 3.6) (drill 1.2) (layers *.Cu *.Mask) (roundrect_rratio 0.1388888889)
       (net 2 "GND") (pinfunction "Pin_1") (pintype "passive"))
     (pad "2" thru_hole oval (at 5.08 0) (size 1.8 3.6) (drill 1.2) (layers *.Cu *.Mask)
@@
     (fp_line (start 1.6 -0.8) (end 1.6 0.8) (layer "F.Fab") (width 0.1))
     (fp_line (start -1.6 0.8) (end -1.6 -0.8) (layer "F.Fab") (width 0.1))
-    (pad "1" smd roundrect (at -1.4625 0) (size 1.125 1.75) (layers "F.Cu" "F.Paste" "F.Mask") (roundrect_rratio 0.222222)
+    (pad "1" smd roundrect (at -1.4625 0) (size 1.125 1.75) (layers "F.Cu" "F.Paste" "F.Mask") (roundrect_rratio 0.2222222222)
       (net 29 "+5V") (pintype "passive"))
-    (pad "2" smd roundrect (at 1.4625 0) (size 1.125 1.75) (layers "F.Cu" "F.Paste" "F.Mask") (roundrect_rratio 0.222222)
+    (pad "2" smd roundrect (at 1.4625 0) (size 1.125 1.75) (layers "F.Cu" "F.Paste" "F.Mask") (roundrect_rratio 0.2222222222)
       (net 2 "GND") (pintype "passive"))
     (model "${KICAD6_3DMODEL_DIR}/Resistor_SMD.3dshapes/R_1206_3216Metric.wrl"
@@
     (fp_line (start -1.6 0.8) (end -1.6 -0.8) (layer "F.Fab") (width 0.1))
     (fp_line (start 1.6 0.8) (end -1.6 0.8) (layer "F.Fab") (width 0.1))
-    (pad "1" smd roundrect (at -1.4625 0) (size 1.125 1.75) (layers "F.Cu" "F.Paste" "F.Mask") (roundrect_rratio 0.222222)
+    (pad "1" smd roundrect (at -1.4625 0) (size 1.125 1.75) (layers "F.Cu" "F.Paste" "F.Mask") (roundrect_rratio 0.2222222222)
       (net 29 "+5V") (pintype "passive"))
-    (pad "2" smd roundrect (at 1.4625 0) (size 1.125 1.75) (layers "F.Cu" "F.Paste" "F.Mask") (roundrect_rratio 0.222222)
+    (pad "2" smd roundrect (at 1.4625 0) (size 1.125 1.75) (layers "F.Cu" "F.Paste" "F.Mask") (roundrect_rratio 0.2222222222)
       (net 2 "GND") (pintype "passive"))
     (model "${KICAD6_3DMODEL_DIR}/Resistor_SMD.3dshapes/R_1206_3216Metric.wrl"
@@
     (fp_line (start -1.6 -0.8) (end 1.6 -0.8) (layer "F.Fab") (width 0.1))
     (fp_line (start -1.6 0.8) (end -1.6 -0.8) (layer "F.Fab") (width 0.1))
-    (pad "1" smd roundrect (at -1.4625 0) (size 1.125 1.75) (layers "F.Cu" "F.Paste" "F.Mask") (roundrect_rratio 0.222222)
+    (pad "1" smd roundrect (at -1.4625 0) (size 1.125 1.75) (layers "F.Cu" "F.Paste" "F.Mask") (roundrect_rratio 0.2222222222)
       (net 29 "+5V") (pintype "passive"))
-    (pad "2" smd roundrect (at 1.4625 0) (size 1.125 1.75) (layers "F.Cu" "F.Paste" "F.Mask") (roundrect_rratio 0.222222)
+    (pad "2" smd roundrect (at 1.4625 0) (size 1.125 1.75) (layers "F.Cu" "F.Paste" "F.Mask") (roundrect_rratio 0.2222222222)
       (net 2 "GND") (pintype "passive"))
     (model "${KICAD6_3DMODEL_DIR}/Resistor_SMD.3dshapes/R_1206_3216Metric.wrl"
@@
     (fp_line (start -1.6 -0.8) (end 1.6 -0.8) (layer "F.Fab") (width 0.1))
     (fp_line (start 1.6 0.8) (end -1.6 0.8) (layer "F.Fab") (width 0.1))
-    (pad "1" smd roundrect (at -1.4625 0 180) (size 1.125 1.75) (layers "F.Cu" "F.Paste" "F.Mask") (roundrect_rratio 0.222222)
+    (pad "1" smd roundrect (at -1.4625 0 180) (size 1.125 1.75) (layers "F.Cu" "F.Paste" "F.Mask") (roundrect_rratio 0.2222222222)
       (net 30 "VDD") (pintype "passive"))
-    (pad "2" smd roundrect (at 1.4625 0 180) (size 1.125 1.75) (layers "F.Cu" "F.Paste" "F.Mask") (roundrect_rratio 0.222222)
+    (pad "2" smd roundrect (at 1.4625 0 180) (size 1.125 1.75) (layers "F.Cu" "F.Paste" "F.Mask") (roundrect_rratio 0.2222222222)
       (net 2 "GND") (pintype "passive"))
     (model "${KICAD6_3DMODEL_DIR}/Resistor_SMD.3dshapes/R_1206_3216Metric.wrl"
@@
     (fp_line (start 1.6 0.8) (end 1.6 -0.8) (layer "B.Fab") (width 0.1))
     (fp_line (start -1.6 0.8) (end 1.6 0.8) (layer "B.Fab") (width 0.1))
-    (pad "1" smd roundrect (at -1.4625 0 90) (size 1.125 1.75) (layers "B.Cu" "B.Paste" "B.Mask") (roundrect_rratio 0.222222)
+    (pad "1" smd roundrect (at -1.4625 0 90) (size 1.125 1.75) (layers "B.Cu" "B.Paste" "B.Mask") (roundrect_rratio 0.2222222222)
       (net 1 "+3V3") (pintype "passive"))
-    (pad "2" smd roundrect (at 1.4625 0 90) (size 1.125 1.75) (layers "B.Cu" "B.Paste" "B.Mask") (roundrect_rratio 0.222222)
+    (pad "2" smd roundrect (at 1.4625 0 90) (size 1.125 1.75) (layers "B.Cu" "B.Paste" "B.Mask") (roundrect_rratio 0.2222222222)
       (net 2 "GND") (pintype "passive"))
     (model "${KICAD6_3DMODEL_DIR}/Resistor_SMD.3dshapes/R_1206_3216Metric.wrl"
@@
     (fp_line (start -1.6 -0.8) (end -1.6 0.8) (layer "B.Fab") (width 0.1))
     (fp_line (start 1.6 -0.8) (end -1.6 -0.8) (layer "B.Fab") (width 0.1))
-    (pad "1" smd roundrect (at -1.4625 0 90) (size 1.125 1.75) (layers "B.Cu" "B.Paste" "B.Mask") (roundrect_rratio 0.222222)
+    (pad "1" smd roundrect (at -1.4625 0 90) (size 1.125 1.75) (layers "B.Cu" "B.Paste" "B.Mask") (roundrect_rratio 0.2222222222)
       (net 1 "+3V3") (pintype "passive"))
-    (pad "2" smd roundrect (at 1.4625 0 90) (size 1.125 1.75) (layers "B.Cu" "B.Paste" "B.Mask") (roundrect_rratio 0.222222)
+    (pad "2" smd roundrect (at 1.4625 0 90) (size 1.125 1.75) (layers "B.Cu" "B.Paste" "B.Mask") (roundrect_rratio 0.2222222222)
       (net 2 "GND") (pintype "passive"))
     (model "${KICAD6_3DMODEL_DIR}/Resistor_SMD.3dshapes/R_1206_3216Metric.wrl"
@@
     (effects (font (size 1 1) (thickness 0.15)))
   )
+  (gr_text "JLCJLCJLCJLC" (at 185.8 84 90) (layer "F.SilkS")
+    (effects (font (size 1 1) (thickness 0.15)))
+  )
